Commit message: Spawns two robots models (the same)

File: urdf/torpedoes.xacro (robot description, xacro)
@@ -5,5 +5,5 @@
 <link name="torpedoes">
     <visual>
-        <origin xyz="1 1 1" rpy="0.0 0.0 0.0"/>
+        <origin xyz="0 0 0" rpy="0.0 0.0 0.0"/>
         <geometry>
             <mesh filename="${visual_mesh_file}" scale="0.001 0.001 0.001" />
