Commit message: Se exportan dos modelos diferentes sin errores

File: urdf/shooter.xacro (robot description, xacro)
@@ -13,5 +13,5 @@
       <origin xyz="0 0 0" rpy="0 0 0"/>
       <geometry>
-        <box size="1 1 1"/>
+        <box size="0.01 0.01 0.01"/>
       </geometry>
     </collision>

File: urdf/torpedoes.xacro (robot description, xacro)
@@ -5,5 +5,5 @@
 <link name="torpedoes">
     <visual>
-        <origin xyz="0 0 0" rpy="0.0 0.0 0.0"/>
+        <origin xyz="-10 -10 0" rpy="0.0 0.0 1.57075"/>
         <geometry>
             <mesh filename="${visual_mesh_file}" scale="0.001 0.001 0.001" />
@@ -14,5 +14,5 @@
       <origin xyz="0 0 0" rpy="0 0 0"/>
       <geometry>
-        <box size="1 1 1"/>
+        <box size="0.07 0.07 0.07"/>
       </geometry>
     </collision>

Commit message: inician macros

File: urdf/shooter.xacro (robot description, xacro)
@@ -1,5 +1,5 @@
 <?xml version="1.0"?>
 <robot name="shooter" xmlns:xacro="http://www.ros.org/wiki/xacro">
-<xacro:property name="visual_mesh_file" value="file://$(find shooter_description)/meshes/shooter.dae" />
+<xacro:property name="visual_mesh_file" value="file://$(find shooter_description)/meshes/base_simulacion_origen_corregido.dae" />
 <link name="base_link">
     <visual>

File: urdf/torpedoes.xacro (robot description, xacro)
@@ -2,8 +2,8 @@
 <robot name="torpedoes" xmlns:xacro="http://www.ros.org/wiki/xacro">
 <!-- Introducir meshes -->
-<xacro:property name="visual_mesh_file" value="file://$(find shooter_description)/meshes/torpedoes.dae" />
+<xacro:property name="visual_mesh_file" value="file://$(find shooter_description)/meshes/Torpedo_simulacion_origen_corregido.dae" />
 <link name="torpedoes">
     <visual>
-        <origin xyz="-10 -10 0" rpy="0.0 0.0 1.57075"/>
+        <origin xyz="0.085 0 0" rpy="0.0 0.0 1.57075"/>
         <geometry>
             <mesh filename="${visual_mesh_file}" scale="0.001 0.001 0.001" />
