Commit message: Spawns two models, but they are on 0 0 0

File: urdf/macro_torpedoes.xacro (robot description, xacro)
@@ -1,4 +1,31 @@
-<?xml version="1.0">
+<?xml version="1.0"?>
 <robot name="macro_torpedoes" xmlns:xacro="http://www.ros.org/wiki/xacro">
-<xacro:torpedoes_macro robot_namespace="${namespace" torpedoes_id="0">
+<!-- Introducir meshes -->
+<xacro:property name="visual_mesh_file" value="file://$(find shooter_description)/meshes/Torpedo_simulacion_origen_corregido.dae" />
+<xacro:macro name="macro_torpedoes" params="id">
+<!-- <origin xyz="0.085 (0 -0.085) 0 0" rpy="0.0 0.0 1.57075"/> -->
+<link name="torpedoes_${id}">
+    <visual>
+        <origin xyz="0.085 0 0" rpy="0.0 0.0 1.57075"/>
+        <geometry>
+            <mesh filename="${visual_mesh_file}" scale="0.001 0.001 0.001" />
+        </geometry>
+    </visual>
+        <!-- Se deben cambiar los parametros reales-->
+    <collision>
+      <origin xyz="0 0 0" rpy="0 0 0"/>
+      <geometry>
+        <box size="0.07 0.07 0.07"/>
+      </geometry>
+    </collision>
+    <inertial>
+      <origin xyz="0 0 0" rpy="0 0 0"/>
+      <mass value="1"/>
+      <inertia
+        ixx="1.0" ixy="0.0" ixz="0.0"
+        iyy="1.0" iyz="0.0"
+        izz="1.0"/>
+    </inertial>
+</link>
+</xacro:macro>
 </robot>

File: urdf/shooter.xacro (robot description, xacro)
@@ -4,5 +4,5 @@
 <link name="base_link">
     <visual>
-        <origin xyz="0.0 0.0 0.0" rpy="0.0 0.0 0.0"/>
+        <origin xyz="0.0 0.0 0.1" rpy="0.0 0.0 0.0"/>
         <geometry>
             <mesh filename="${visual_mesh_file}" scale="0.001 0.001 0.001"/>

File: urdf/torpedoes.xacro (robot description, xacro)
@@ -1,9 +1,10 @@
 <?xml version="1.0"?>
-<robot name="torpedoes" xmlns:xacro="http://www.ros.org/wiki/xacro">
+<robot name="macro_torpedoes" xmlns:xacro="http://www.ros.org/wiki/xacro">
 <!-- Introducir meshes -->
 <xacro:property name="visual_mesh_file" value="file://$(find shooter_description)/meshes/Torpedo_simulacion_origen_corregido.dae" />
+<!-- <origin xyz="0.085 (0 -0.085) 0 0" rpy="0.0 0.0 1.57075"/> -->
 <link name="torpedoes">
     <visual>
-        <origin xyz="0.085 0 0" rpy="0.0 0.0 1.57075"/>
+        <origin xyz="0 0 0" rpy="0.0 0.0 1.57075"/>
         <geometry>
             <mesh filename="${visual_mesh_file}" scale="0.001 0.001 0.001" />

Commit message: Correct usage of macro and changed origin in one shooter. Spawn Robots: shooter, torpedoes_1

File: urdf/macro_torpedoes.xacro (robot description, xacro)
@@ -3,9 +3,9 @@
 <!-- Introducir meshes -->
 <xacro:property name="visual_mesh_file" value="file://$(find shooter_description)/meshes/Torpedo_simulacion_origen_corregido.dae" />
-<xacro:macro name="macro_torpedoes" params="id">
+<xacro:macro name="macro_torpedoes" params="id *origin">
 <!-- <origin xyz="0.085 (0 -0.085) 0 0" rpy="0.0 0.0 1.57075"/> -->
 <link name="torpedoes_${id}">
     <visual>
-        <origin xyz="0.085 0 0" rpy="0.0 0.0 1.57075"/>
+        <xacro:insert_block name="origin"/>
         <geometry>
             <mesh filename="${visual_mesh_file}" scale="0.001 0.001 0.001" />

File: urdf/shooter.xacro (robot description, xacro)
@@ -9,5 +9,4 @@
         </geometry>
     </visual>
-    <!-- Se deben cambiar los parametros reales-->
     <collision>
       <origin xyz="0 0 0" rpy="0 0 0"/>

File: urdf/torpedoes.xacro (robot description, xacro)
@@ -1,7 +1,6 @@
 <?xml version="1.0"?>
 <robot name="macro_torpedoes" xmlns:xacro="http://www.ros.org/wiki/xacro">
-<!-- Introducir meshes -->
+<!-- Introducir meshes
 <xacro:property name="visual_mesh_file" value="file://$(find shooter_description)/meshes/Torpedo_simulacion_origen_corregido.dae" />
-<!-- <origin xyz="0.085 (0 -0.085) 0 0" rpy="0.0 0.0 1.57075"/> -->
 <link name="torpedoes">
     <visual>
@@ -11,5 +10,4 @@
         </geometry>
     </visual>
-        <!-- Se deben cambiar los parametros reales-->
     <collision>
       <origin xyz="0 0 0" rpy="0 0 0"/>
@@ -26,4 +24,8 @@
         izz="1.0"/>
     </inertial>
-</link>
+</link -->
+<xacro:include filename="$(find shooter_description)/urdf/macro_torpedoes.xacro"/>
+<xacro:macro_torpedoes id="1">
+  <origin xyz="1 1 1" rpy="0.0 0.0 1.5757"/>
+</xacro:macro_torpedoes>
 </robot>

Commit message: Correct positioning of shooter and both torpedoes. The collision boxes do not allow torpedoes inside shooter

File: urdf/macro_torpedoes.xacro (robot description, xacro)
@@ -16,5 +16,5 @@
       <origin xyz="0 0 0" rpy="0 0 0"/>
       <geometry>
-        <box size="0.07 0.07 0.07"/>
+        <box size="0.01 0.01 0.01"/>
       </geometry>
     </collision>

File: urdf/shooter.xacro (robot description, xacro)
@@ -1,4 +1,5 @@
 <?xml version="1.0"?>
 <robot name="shooter" xmlns:xacro="http://www.ros.org/wiki/xacro">
+085
 <xacro:property name="visual_mesh_file" value="file://$(find shooter_description)/meshes/base_simulacion_origen_corregido.dae" />
 <link name="base_link">
@@ -12,5 +13,5 @@
       <origin xyz="0 0 0" rpy="0 0 0"/>
       <geometry>
-        <box size="0.01 0.01 0.01"/>
+        <box size="0.001 0.001 0.001"/>
       </geometry>
     </collision>

File: urdf/torpedoes_1.xacro (robot description, xacro)
@@ -1,8 +1,8 @@
 <?xml version="1.0"?>
-<robot name="macro_torpedoes" xmlns:xacro="http://www.ros.org/wiki/xacro">
+<robot name="torpedoes_2" xmlns:xacro="http://www.ros.org/wiki/xacro">
 <!-- Incluir el archivo de la macro -->
 <xacro:include filename="$(find shooter_description)/urdf/macro_torpedoes.xacro"/>
-<xacro:macro_torpedoes id="1">
-  <origin xyz="0.085 0 0" rpy="0.0 0.0 1.5757"/>
+<xacro:macro_torpedoes id="2">
+  <origin xyz="-0.085 0 0" rpy="0.0 0.0 1.5757"/>
 </xacro:macro_torpedoes>
 </robot>

Commit message: The three models are COMPLETELY and correctly imported into gazebo

File: urdf/macro_torpedoes.xacro (robot description, xacro)
@@ -3,4 +3,5 @@
 <!-- Introducir meshes -->
 <xacro:property name="visual_mesh_file" value="file://$(find shooter_description)/meshes/Torpedo_simulacion_origen_corregido.dae" />
+<xacro:property name="collision_mesh_file" value="file://$(find shooter_description)/meshes/Torpedo_simulacion_rebajado.STL" />
 <xacro:macro name="macro_torpedoes" params="id *origin">
 <!-- <origin xyz="0.085 (0 -0.085) 0 0" rpy="0.0 0.0 1.57075"/> -->
@@ -14,11 +15,13 @@
         <!-- Se deben cambiar los parametros reales-->
     <collision>
-      <origin xyz="0 0 0" rpy="0 0 0"/>
+      <xacro:insert_block name="origin"/>
       <geometry>
-        <box size="0.01 0.01 0.01"/>
+        <!--No mover el collision box-->
+        <box size="0.05 0.05 0.15"/>
+        <!-- mesh filename="${collision_mesh_file}" scale="0.001 0.001 0.001" / -->
       </geometry>
     </collision>
     <inertial>
-      <origin xyz="0 0 0" rpy="0 0 0"/>
+      <xacro:insert_block name="origin"/>
       <mass value="1"/>
       <inertia

File: urdf/shooter.xacro (robot description, xacro)
@@ -2,7 +2,8 @@
 <robot name="shooter" xmlns:xacro="http://www.ros.org/wiki/xacro">
 <xacro:property name="visual_mesh_file" value="file://$(find shooter_description)/meshes/base_simulacion_origen_corregido.dae" />
+<xacro:property name="collision_mesh_file" value="file://$(find shooter_description)/meshes/base_simulacion.STL"/>
 <link name="base_link">
     <visual>
-        <origin xyz="0.0 0.0 0.1" rpy="0.0 0.0 0.0"/>
+        <origin xyz="0.0 0.0 0.23" rpy="0.0 0.0 0.0"/>
         <geometry>
             <mesh filename="${visual_mesh_file}" scale="0.001 0.001 0.001"/>
@@ -10,12 +11,13 @@
     </visual>
     <collision>
-      <origin xyz="0 0 0" rpy="0 0 0"/>
+      <origin xyz="0 0 0.23" rpy="0 0 0"/>
       <geometry>
-        <box size="0.001 0.001 0.001"/>
+        <box size="0.1 0.1 0.1"/>
+        <!-- mesh filename="${collision_mesh_file}" scale="0.001 0.001 0.001" / -->
       </geometry>
     </collision>
     <inertial>
-      <origin xyz="0 0 0" rpy="0 0 0"/>
-      <mass value="1"/>
+      <origin xyz="0 0 0.2" rpy="0 0 0"/>
+      <mass value="10"/>
       <inertia
         ixx="1.0" ixy="0.0" ixz="0.0"

File: urdf/torpedoes_1.xacro (robot description, xacro)
@@ -4,4 +4,5 @@
 <xacro:include filename="$(find shooter_description)/urdf/macro_torpedoes.xacro"/>
 <xacro:macro_torpedoes id="2">
+  <!--<origin xyz="-0.085 0 0" rpy="0.0 0.0 1.5757"/>-->
   <origin xyz="-0.085 0 0" rpy="0.0 0.0 1.5757"/>
 </xacro:macro_torpedoes>
